Commit message: multirobot urdf experiments

File: examples/multiPointRobot.urdf (robot description, URDF)
Before this commit: robot pointRobot, 14 links, 13 joints
Links:
- removed link holder_right
Joints:
- removed joint base_to_holder

Commit message: PPO_v1

File: examples/multiPointRobot.urdf (robot description, URDF)
Before this commit: robot pointRobot, 13 links, 12 joints
Joints:
- joint mobile_joint_x_1: axis 1 0 0 -> 0 0 1
