Commit message: changes to ppo

File: examples/loadPointRobot.urdf (robot description, URDF)
Before this commit: robot pointRobot, 11 links, 10 joints
Links:
- link big_planck: geometry collision box size=0.5 0.5 0.05; visual box size=0.5 0.5 0.05
- link holder_left: mass None -> 0.1
- link holder_right: mass None -> 0.1
- link holder_top: mass None -> 0.1

Commit message: changed the robot added two inplace holders

File: examples/loadPointRobot.urdf (robot description, URDF)
Before this commit: robot pointRobot, 11 links, 10 joints
Links:
- added link holder_left_top, mass 0.1; collision box size=0.1 0.7 0.3; visual box size=0.1 0.7 0.3
- added link holder_right_top, mass 0.1; collision box size=0.1 0.7 0.3; visual box size=0.1 0.7 0.3
Joints:
- added joint planckt_to_holder_left_top: type fixed, parent big_planck, child holder_left_top, origin xyz=-0.23 0.0 0.15 rpy=0 0 0
- added joint planckt_to_holder_right_top: type fixed, parent big_planck, child holder_right_top, origin xyz=0.23 0.0 0.15 rpy=0 0 0
