Commit message: evolution_strategies and a passage environment added

File: examples/block.urdf (robot description, URDF)
Before this commit: robot block_2, 1 links, 0 joints
Links:
- link block_2_base_link: mass 2.00 -> 5.00

Commit message: working erl+ppo

File: examples/block.urdf (robot description, URDF)
Before this commit: robot block_2, 1 links, 0 joints
Links:
- link block_2_base_link: mass 5.00 -> 2.50

File: examples/loadPointRobot.urdf (robot description, URDF)
Before this commit: robot pointRobot, 13 links, 12 joints
Links:
- link base_link_1: geometry collision cylinder length=0.1 radius=0.3; visual cylinder length=0.1 radius=0.3
- link big_planck: geometry collision box size=0.8 0.8 0.05; visual box size=0.7 0.7 0.05
